Commit message: remove model dependency from controlit_moom controlit_models package

File: Sandboxes/dreamer_viz/robot/dreamer_ltw.urdf (robot description, URDF)
Before this commit: robot dreamer, 47 links, 46 joints
Links:
- link eye_pitch_link: geometry collision box size=0.01 0.01 0.01; visual mesh filename=package://dreamer_viz/models/dreamer/meka_description/meshe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
- link l_gripper_l_finger_link: geometry collision mesh filename=package://dreamer_viz/models/dreamer/meka_description/meshe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; visual mesh filename=package://dreamer_viz/models/dreamer/meka_description/meshe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
- link l_gripper_l_finger_tip_link: geometry collision mesh filename=package://dreamer_viz/models/dreamer/meka_description/meshe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; visual mesh filename=package://dreamer_viz/models/dreamer/meka_description/meshe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
- link l_gripper_palm_link: geometry collision mesh filename=package://dreamer_viz/models/dreamer/meka_description/meshe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; visual mesh filename=package://dreamer_viz/models/dreamer/meka_description/meshe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
- link l_gripper_r_finger_link: geometry collision mesh filename=package://dreamer_viz/models/dreamer/meka_description/meshe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; visual mesh filename=package://dreamer_viz/models/dreamer/meka_description/meshe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
- link l_gripper_r_finger_tip_link: geometry collision mesh filename=package://dreamer_viz/models/dreamer/meka_description/meshe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; visual mesh filename=package://dreamer_viz/models/dreamer/meka_description/meshe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
- link left_elbow_link: geometry collision mesh filename=package://dreamer_viz/models/dreamer/meka_description/meshe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; visual mesh filename=package://dreamer_viz/models/dreamer/meka_description/meshe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
- link left_eye_yaw_link: geometry collision mesh filename=package://dreamer_viz/models/dreamer/meka_description/meshe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; visual mesh filename=package://dreamer_viz/models/dreamer/meka_description/meshe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
- link left_shoulder_abductor_link: geometry collision mesh filename=package://dreamer_viz/models/dreamer/meka_description/meshe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; visual mesh filename=package://dreamer_viz/models/dreamer/meka_description/meshe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
- link left_shoulder_extensor_link: geometry collision mesh filename=package://dreamer_viz/models/dreamer/meka_description/meshe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; visual mesh filename=package://dreamer_viz/models/dreamer/meka_description/meshe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
- link left_shoulder_rotator_link: geometry collision mesh filename=package://dreamer_viz/models/dreamer/meka_description/meshe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; visual mesh filename=package://dreamer_viz/models/dreamer/meka_description/meshe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
- link left_wrist_pitch_link: geometry collision box size=0.01 0.01 0.01; visual mesh filename=package://dreamer_viz/models/dreamer/meka_description/meshe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
- link left_wrist_rotator_link: geometry collision mesh filename=package://dreamer_viz/models/dreamer/meka_description/meshe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; visual mesh filename=package://dreamer_viz/models/dreamer/meka_description/meshe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
- link left_wrist_yaw_link: geometry collision mesh filename=package://dreamer_viz/models/dreamer/meka_description/meshe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; visual mesh filename=package://dreamer_viz/models/dreamer/meka_description/meshe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
- link lower_neck_pitch_link: geometry collision mesh filename=package://dreamer_viz/models/dreamer/meka_description/meshe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; visual mesh filename=package://dreamer_viz/models/dreamer/meka_description/meshe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
- link palm: geometry collision mesh filename=package://dreamer_viz/models/dreamer/meka_description/meshe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; visual mesh filename=package://dreamer_viz/models/dreamer/meka_description/meshe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
- link panplate_link: geometry collision mesh filename=package://dreamer_viz/models/dreamer/meka_description/meshe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; visual mesh filename=package://dreamer_viz/models/dreamer/meka_description/meshe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
- link right_elbow_link: geometry collision mesh filename=package://dreamer_viz/models/dreamer/meka_description/meshe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; visual mesh filename=package://dreamer_viz/models/dreamer/meka_description/meshe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
- link right_eye_yaw_link: geometry collision mesh filename=package://dreamer_viz/models/dreamer/meka_description/meshe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; visual mesh filename=package://dreamer_viz/models/dreamer/meka_description/meshe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
- link right_middle_finger_dip_link: geometry collision mesh filename=package://dreamer_viz/models/dreamer/meka_description/meshe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; visual mesh filename=package://dreamer_viz/models/dreamer/meka_description/meshe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
- link right_middle_finger_mcp_link: geometry collision mesh filename=package://dreamer_viz/models/dreamer/meka_description/meshe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; visual mesh filename=package://dreamer_viz/models/dreamer/meka_description/meshe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
- link right_middle_finger_pip_link: geometry collision mesh filename=package://dreamer_viz/models/dreamer/meka_description/meshe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; visual mesh filename=package://dreamer_viz/models/dreamer/meka_description/meshe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
- link right_pinky_dip_link: geometry collision mesh filename=package://dreamer_viz/models/dreamer/meka_description/meshe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; visual mesh filename=package://dreamer_viz/models/dreamer/meka_description/meshe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
- link right_pinky_mcp: geometry collision mesh filename=package://dreamer_viz/models/dreamer/meka_description/meshe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; visual mesh filename=package://dreamer_viz/models/dreamer/meka_description/meshe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
- link right_pinky_pip: geometry collision mesh filename=package://dreamer_viz/models/dreamer/meka_description/meshe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; visual mesh filename=package://dreamer_viz/models/dreamer/meka_description/meshe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
- link right_pointer_finger_dip_link: geometry collision mesh filename=package://dreamer_viz/models/dreamer/meka_description/meshe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; visual mesh filename=package://dreamer_viz/models/dreamer/meka_description/meshe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
- link right_pointer_finger_mcp_link: geometry collision mesh filename=package://dreamer_viz/models/dreamer/meka_description/meshe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; visual mesh filename=package://dreamer_viz/models/dreamer/meka_description/meshe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
- link right_pointer_finger_pip: geometry collision mesh filename=package://dreamer_viz/models/dreamer/meka_description/meshe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; visual mesh filename=package://dreamer_viz/models/dreamer/meka_description/meshe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
- link right_shoulder_abductor_link: geometry collision mesh filename=package://dreamer_viz/models/dreamer/meka_description/meshe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; visual mesh filename=package://dreamer_viz/models/dreamer/meka_description/meshe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
- link right_shoulder_extensor_link: geometry collision mesh filename=package://dreamer_viz/models/dreamer/meka_description/meshe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; visual mesh filename=package://dreamer_viz/models/dreamer/meka_description/meshe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
- link right_shoulder_rotator_link: geometry collision mesh filename=package://dreamer_viz/models/dreamer/meka_description/meshe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; visual mesh filename=package://dreamer_viz/models/dreamer/meka_description/meshe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
- link right_thumb_cmc_link: geometry collision mesh filename=package://dreamer_viz/models/dreamer/meka_description/meshe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; visual mesh filename=package://dreamer_viz/models/dreamer/meka_description/meshe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 scale=1 1 1
- link right_thumb_ip_link: geometry collision mesh filename=package://dreamer_viz/models/dreamer/meka_description/meshe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; visual mesh filename=package://dreamer_viz/models/dreamer/meka_description/meshe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
- link right_thumb_mcp_link: geometry collision mesh filename=package://dreamer_viz/models/dreamer/meka_description/meshe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; visual mesh filename=package://dreamer_viz/models/dreamer/meka_description/meshe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
- link right_wrist_pitch_link: geometry collision box size=0.01 0.01 0.01; visual mesh filename=package://dreamer_viz/models/dreamer/meka_description/meshe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
- link right_wrist_rotator_link: geometry collision mesh filename=package://dreamer_viz/models/dreamer/meka_description/meshe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; visual mesh filename=package://dreamer_viz/models/dreamer/meka_description/meshe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
- link right_wrist_yaw_link: geometry collision mesh filename=package://dreamer_viz/models/dreamer/meka_description/meshe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; visual mesh filename=package://dreamer_viz/models/dreamer/meka_description/meshe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
- link torso_lower_pitch_link: geometry collision mesh filename=package://dreamer_viz/models/dreamer/meka_description/meshe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; visual mesh filename=package://dreamer_viz/models/dreamer/meka_description/meshe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
- link torso_upper_pitch_link: geometry collision mesh filename=package://dreamer_viz/models/dreamer/meka_description/meshe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; visual mesh filename=package://dreamer_viz/models/dreamer/meka_description/meshe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
- link torso_yaw_link: geometry collision mesh filename=package://dreamer_viz/models/dreamer/meka_description/meshe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; visual mesh filename=package://dreamer_viz/models/dreamer/meka_description/meshe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
- link upper_neck_pitch_link: geometry collision mesh filename=package://dreamer_viz/models/dreamer/meka_description/meshe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; visual mesh filename=package://dreamer_viz/models/dreamer/meka_description/meshe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
- link upper_neck_roll_link: geometry collision box size=0.01 0.01 0.01; visual mesh filename=package://dreamer_viz/models/dreamer/meka_description/meshe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
- link upper_neck_yaw_link: geometry collision box size=0.01 0.01 0.01; visual mesh filename=package://dreamer_viz/models/dreamer/meka_description/meshe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
